File: Internal_Expander/KiCad/VIC20_Internal_Expander.kicad_pcb (KiCad board)
At the start: 2 copper layers, 85 x 58 mm, 12 parts, among them J1 UD2, J2 UE2, J3 UD6, J4 UE6, J5 SW, J6 Signals, U1 6264 RAM, U2 GAL16V8, U3 2764 ROM

Commit message: Further design
Parts:
- moved J3 49.4 mm to (125.4, 32.6)
- moved G*** 46.7 mm to (111.4, 35.6)
- moved J4 41.6 mm to (125.4, 62.6)
- moved C1 38.7 mm to (97.4, 47.6), turned to 90 degrees
- moved J1 34.4 mm to (55.4, 32.6)
- moved J2 34.4 mm to (55.4, 62.6)
- moved R1 34.4 mm to (69.7, 43.6)
- moved U3 34.4 mm to (70.1, 49.7)
- moved U1 34.4 mm to (104.4, 49.5)
- moved U2 34.4 mm to (91.1, 59.2)
- moved J5 25.8 mm to (72.4, 37.6)
- moved J6 25.2 mm to (95.0, 37.6)
Connections:
- J1 pad 1: VA6 -> unconnected-(J1-Pin_1-Pad1)
- J1 pad 10: VR/W -> unconnected-(J1-Pin_10-Pad10)
- J1 pad 11: BD3 -> unconnected-(J1-Pin_11-Pad11)
- J1 pad 15: VA9 -> unconnected-(J1-Pin_15-Pad15)
- J1 pad 16: VA8 -> unconnected-(J1-Pin_16-Pad16)
- J1 pad 2: VA5 -> unconnected-(J1-Pin_2-Pad2)
- J1 pad 3: VA4 -> unconnected-(J1-Pin_3-Pad3)
- J1 pad 4: VA3 -> unconnected-(J1-Pin_4-Pad4)
- J1 pad 5: VA0 -> unconnected-(J1-Pin_5-Pad5)
- J1 pad 6: VA1 -> unconnected-(J1-Pin_6-Pad6)
- J1 pad 7: VA2 -> unconnected-(J1-Pin_7-Pad7)
- J2 pad 17: VA7 -> unconnected-(J2-Pin_17-Pad17)
- J3 pad 1: VA6 -> unconnected-(J3-Pin_1-Pad1)
- J3 pad 10: VR/W -> unconnected-(J3-Pin_10-Pad10)
- J3 pad 11: BD3 -> unconnected-(J3-Pin_11-Pad11)
- J3 pad 12: BD2 -> unconnected-(J3-Pin_12-Pad12)
- J3 pad 13: BD1 -> unconnected-(J3-Pin_13-Pad13)
- J3 pad 14: BD0 -> unconnected-(J3-Pin_14-Pad14)
- J3 pad 15: VA9 -> unconnected-(J3-Pin_15-Pad15)
- J3 pad 16: VA8 -> unconnected-(J3-Pin_16-Pad16)
- J3 pad 17: VA7 -> unconnected-(J3-Pin_17-Pad17)
- J3 pad 2: VA5 -> unconnected-(J3-Pin_2-Pad2)
- J3 pad 3: VA4 -> unconnected-(J3-Pin_3-Pad3)
- J3 pad 4: VA3 -> unconnected-(J3-Pin_4-Pad4)
- J3 pad 5: VA0 -> unconnected-(J3-Pin_5-Pad5)
- J3 pad 6: VA1 -> unconnected-(J3-Pin_6-Pad6)
- J3 pad 7: VA2 -> unconnected-(J3-Pin_7-Pad7)
Routing:
- net VA2: track 0.00 -> 120.0 mm, vias 0 -> 3
- net BD0: track 1.56 -> 117.4 mm, vias 0 -> 2
- net VA7: track 0.00 -> 107.9 mm, vias 0 -> 2
- net VA9: track 17.7 -> 114.4 mm, vias 0 -> 3
- net BD7: track 0.00 -> 83.6 mm, vias 0 -> 2
- net VA5: track 23.3 -> 102.8 mm, vias 0 -> 2
- net VA0: track 1.19 -> 78.2 mm, vias 0 -> 3
- net VA1: track 0.00 -> 75.7 mm, vias 0 -> 1
- net VA8: track 17.7 -> 92.1 mm, vias 0 -> 4
- net VA10: track 0.00 -> 72.6 mm, vias 0 -> 1
- net BD5: track 0.00 -> 72.0 mm, vias 0 -> 3
- net BD2: track 30.7 -> 102.5 mm
- net BD1: track 30.5 -> 101.4 mm
- net VA12: track 0.00 -> 70.1 mm, vias 0 -> 1
- net VR/W: track 13.9 -> 82.9 mm, vias 0 -> 1
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Other:
- board size 85 x 58 mm -> 84 x 60 mm
- board text added: "Internal Super Expander ©2025 Rev. A"
- board text added: "VA10 VA11 VA12 VA13 BLK0 BLK5 Φ2"
- board text removed: "Internal Super Expander ©2025"
- board text removed: "VA10 VA11 VA12 VA13 BLK0 Φ2 BLK5"
