File: Internal_Expander/KiCad/VIC20_Internal_Expander.kicad_sch (KiCad schematic)
At the start: 11 parts, among them J1 UD2, J2 UE2, J3 UD6, J4 UE6, J5 SW, J6 Signals, U1 6264 RAM, U2 GAL16V8, U3 2764 ROM

Commit message: Further design
Connections:
- net BD0: no longer J3.14 (Pin_14)
- net BD1: no longer J3.13 (Pin_13)
- net BD2: no longer J3.12 (Pin_12)
- net BD3: no longer J1.11 (Pin_11), J3.11 (Pin_11)
- net VA0: no longer J1.5 (Pin_5), J3.5 (Pin_5)
- net VA1: no longer J1.6 (Pin_6), J3.6 (Pin_6)
- net VA2: no longer J1.7 (Pin_7), J3.7 (Pin_7)
- net VA3: no longer J1.4 (Pin_4), J3.4 (Pin_4)
- net VA4: no longer J1.3 (Pin_3), J3.3 (Pin_3)
- net VA5: no longer J1.2 (Pin_2), J3.2 (Pin_2)
- net VA6: no longer J1.1 (Pin_1), J3.1 (Pin_1)
- net VA7: no longer J2.17 (Pin_17), J3.17 (Pin_17)
- net VA8: no longer J1.16 (Pin_16), J3.16 (Pin_16)
- net VA9: no longer J1.15 (Pin_15), J3.15 (Pin_15)
- net VR/W: no longer J1.10 (Pin_10), J3.10 (Pin_10)
- no-connect marks 11 -> 38
Other:
- moved on the sheet: C1, J5, J6, R1
