File: Internal_32KB/KiCad/74LS138_Board_BLK/VIC20_Internal_32KB_BLK_Decode.kicad_pcb (KiCad board)
At the start: 2 copper layers, 12 x 24 mm, 3 parts, among them J1 BLK Outputs, J2 BLK Inputs

Commit message: Updates to 32KB board design
Other:
- board text added: "BLK"
- board text added: "VIC-20 BLK Decoder Logic Replacement Brett Hallen, May 2025"
- board text removed: "VIC-20 Internal 32KB RAM Brett Hallen, May 2025"
Changed lines of the file:
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@@
 			(at 0.62 -2.33 0)
 			(layer "F.SilkS")
+			(hide yes)
 			(effects
 				(font
@@
 		)
 		(property "Value" "74LS138"
-			(at 5.62 -2.33 0)
+			(at 6.582156 -2.333789 0)
 			(layer "F.SilkS")
 			(effects
 				(font
-					(size 1 1)
+					(size 0.8 0.8)
 					(thickness 0.15)
 				)
@@
 		(layer "Edge.Cuts")
 	)
-	(gr_text "VIC-20 Internal 32KB RAM\nBrett Hallen, May 2025"
-		(at 74.38 71.1 270)
+	(gr_text "BLK"
+		(at 71.38 50.284961 0)
+		(layer "F.SilkS")
+		(effects
+			(font
+				(size 0.8 0.8)
+				(thickness 0.15)
+				(bold yes)
+			)
+			(justify left bottom)
+		)
+	)
+	(gr_text "VIC-20 BLK Decoder Logic Replacement\nBrett Hallen, May 2025"
+		(at 75.169921 71.15 270)
 		(layer "B.SilkS")
 		(effects
@@
 	)
 	(segment
-		(start 72.38 64.8)
+		(start 74.6801 59.72)
 		(end 74.6801 62.4999)
 		(width 0.2)
-		(layer "F.Cu")
+		(layer "B.Cu")
 		(net 9)
 	)
 	(segment
 		(start 74.6801 62.4999)
-		(end 74.6801 59.72)
-		(width 0.2)
-		(layer "F.Cu")
+		(end 72.38 64.8)
+		(width 0.2)
+		(layer "B.Cu")
 		(net 9)
 	)
