File: Internal_32KB/KiCad/74LS138_Board_RAM/VIC20_Internal_32KB_RAM_Decode.kicad_sch (KiCad schematic)
At the start: 2 parts, among them J1 Signals

Commit message: Updates to 32KB board design
Other:
- title: Commodore VIC-20 BLK0 RAM Expansion, Daughterboard -> Commodore VIC-20 32KB RAM Expansion,RAM Deocder
Changed lines of the file:
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@@
 	(paper "A5")
 	(title_block
-		(title "Commodore VIC-20 BLK0 RAM Expansion, Daughterboard")
-		(date "12-May-2025")
+		(title "Commodore VIC-20 32KB RAM Expansion,RAM Deocder")
+		(date "14-May-2025")
 		(rev "A")
 		(company "Brett Hallen")
 		(comment 1 "www.youtube.com/@Brfff")
 	)
+	(text_box "This board replaces the 74LS138 3-to-8 decoder used for the internal RAM chip select logic.\n\nThe logic will instead be implemented in a GAL on the main RAM board."
+		(exclude_from_sim no)
+		(at 22.86 21.59 0)
+		(size 58.42 11.43)
+		(margins 0.9525 0.9525 0.9525 0.9525)
+		(stroke
+			(width 0)
+			(type solid)
+		)
+		(fill
+			(type none)
+		)
+		(effects
+			(font
+				(size 1.27 1.27)
+			)
+			(justify left top)
+		)
+	)
 	(no_connect
